File: project/hardware.kicad_sch (KiCad schematic)
At the start: 101 parts, among them IC1 ESP32-S3-MINI-1-N8, IC2 STM32L052K8T6, J1 Conn_01x02_Socket, J2 USB-C, J3 ST-Link, J4 Display_OLed, J5 Dig_OUTs, J6 Analog_INs, J7 798-DM3D-SF, Q1 pnp TO-92 BC307, Q2 pnp TO-92 BC307, Q3 pnp TO-92 BC307, Q4 pnp TO-92 BC307, SW1 SW_Push, SW2 SW_Push, U1 USBLC6-2SC6, U2 TPS563200, Y1 ABS07-166-32.768KHZ-T, Y2 ECS-400-10-36B2-CKM-TR

Commit message: load switch e esp_ready status
Parts:
- removed D4, D5, D6, D8: 1N4001, symbol Device:D_Small
- removed D7: 3V3, symbol Device:D_Zener_Small
- removed R30: 1K, Resistor_SMD:R_0402_1005Metric, symbol Device:R_Small
- removed S1, S2: btSwitch, Button_Switch_SMD:Panasonic_EVQPUK_EVQPUB, symbol botao:3-1437565-0
- added D11, D12: RB058L-30DDTE25, Project_Library:DIOM5026X220N, symbol Device:D_Small_Filled
- added D13, D14, D15, D5: D_Zener_Filled, Diode_SMD:D_SOD-123, symbol Device:D_Zener_Filled
- added D7: CDBQR42/43-HF, Diode_SMD:D_0402_1005Metric, symbol Device:D_Small
- added F1: Fuse_Small, Fuse:Fuse_1206_3216Metric, symbol Device:Fuse_Small
- added J10: UART, Connector_PinSocket_2.54mm:PinSocket_1x04_P2.54mm_Vertical, symbol Connector_Generic:Conn_01x04
- added J8: Analog_INs, Connector_Molex:Molex_PicoBlade_53048-0410_1x04_P1.25mm_Horizontal, symbol Connector_Generic:Conn_01x04
- added J9: Dig_OUTs, TerminalBlock:TerminalBlock_bornier-4_P5.08mm, symbol Connector_Generic:Conn_01x04
- added JP1, JP2: SolderJumper_2_Bridged, Jumper:SolderJumper-2_P1.3mm_Bridged_RoundedPad1.0x1.5mm, symbol Jumper:SolderJumper_2_Bridged
- added JP3: SolderJumper_2_Open, Jumper:SolderJumper-2_P1.3mm_Open_RoundedPad1.0x1.5mm, symbol Jumper:SolderJumper_2_Open
- added R40: 10kR, Resistor_SMD:R_0603_1608Metric_Pad0.98x0.95mm_HandSolder, symbol Device:R_Small
- added R41: 1K, Resistor_SMD:R_0402_1005Metric, symbol Device:R_Small
- added SW3, SW4: SW_Push, Button_Switch_SMD:SW_SPST_PTS810, symbol Switch:SW_Push
- added U3: SiP32431DR3, Package_TO_SOT_SMD:SOT-363_SC-70-6, symbol Power_Management:SiP32431DR3
- C5: footprint Capacitor_SMD:C_0402_1005Metric -> Capacitor_SMD:C_0402_1005Metric_Pad0.74x0.62mm_HandSolder
- D1, D2: footprint Connector_PinSocket_1.27mm:PinSocket_1x04_P1.27mm_Vertical_SMD_Pin1Left -> Connector_PinSocket_1.27mm:PinSocket_1x04_P1.27mm_Vertical
- D3: value 1N4001 -> CDBQR42/43-HF; footprint (none) -> Diode_SMD:D_0402_1005Metric
- J1: footprint Connector_PinSocket_2.54mm:PinSocket_2x01_P2.54mm_Vertical_SMD -> Connector_Molex:Molex_KK-254_AE-6410-02A_1x02_P2.54mm_Vertical
- J3: footprint Connector_Molex:Molex_PicoBlade_53048-0410_1x04_P1.25mm_Horizontal -> Connector_PinSocket_2.54mm:PinSocket_1x04_P2.54mm_Vertical
- J5: footprint Connector_Molex:Molex_PicoBlade_53048-0410_1x04_P1.25mm_Horizontal -> TerminalBlock:TerminalBlock_bornier-4_P5.08mm
- R13, R19, R20, R21, R22, R23, R24, R25, R26, R31, R7, R9: footprint Resistor_SMD:R_0201_0603Metric_Pad0.64x0.40mm_HandSolder -> Resistor_SMD:R_0603_1608Metric_Pad0.98x0.95mm_HandSolder
- R17, R18: footprint Resistor_SMD:R_0201_0603Metric_Pad0.64x0.40mm_HandSolder -> Resistor_SMD:R_0402_1005Metric_Pad0.72x0.64mm_HandSolder
- R29: value 1K -> 10K
- R8: footprint Resistor_SMD:R_0402_1005Metric -> Resistor_SMD:R_0402_1005Metric_Pad0.72x0.64mm_HandSolder
- U2: footprint Package_TO_SOT_SMD:SOT-23-6 -> Package_TO_SOT_SMD:SOT-23-6_Handsoldering
Connections:
- net VDA is gone; now on net 3V3: C12.1, C14.1, IC2.5 (VDDA)
- net VDD is gone; now on net 3V3: J3.4 (VCC), J4.2 (VCC), R19.2, R20.2, R21.2, R22.2
- net +12V: now also F1.1; no longer J1.1 (Pin_1)
- net 3V3: now also R29.2, R31.2, D13.2 (A), D14.2 (A), D15.2 (A), D5.2 (A), J10.1 (SWDIO), R40.2; no longer C23.2, IC1.14 (IO10), R29.1, R31.1, R36.2, SW1.2, SW2.2
- net BOOT: now also R29.1, SW1.2; no longer R29.2
- net BOOT0: now also SW3.1
- net CTS_0: now also JP2.2 (B); no longer IC1.33 (IO37)
- net CTS_1: now also JP1.2 (B); no longer IC1.34 (IO38)
- net Dp_SCL: now also J4.4 (SDA); no longer J4.3 (SCL)
- net Dp_SDA: now also J4.3 (SCL); no longer J4.4 (SDA)
- net EN: now also U3.1 (OUT); no longer R31.2
- net GND: now also C23.1, SW1.1, SW2.1, D11.1 (K), D12.1 (K), D13.1 (K), D14.1 (K), D15.1 (K), D5.1 (K), D7.1 (K), JP3.1 (A), R41.1, SW3.2, SW4.1, U3.2 (GND), U3.5 (GND); no longer J1.2 (Pin_2), J4.1 (GND)
- net LED_ESP_B: now also IC1.13 (IO9)
- net LED_ESP_G: now also IC1.12 (IO8)
- net LED_ESP_R: now also IC1.11 (IO7)
- net LED_STM_B: now also IC2.27 (PB4)
- net LED_STM_G: now also IC2.29 (PB6)
- net LED_STM_R: now also IC2.30 (PB7)
- net NRST: now also SW4.2
- net RX_0: now also J10.2 (GND)
- net RX_1: now also J10.4 (VCC)
- net digOut_pin_1: now also IC1.8 (IO4)
- net digOut_pin_2: now also IC1.7 (IO3)
- net digOut_pin_3: now also IC1.6 (IO2)
- net digOut_pin_4: now also IC1.5 (IO1)
- net ESP_EN: now reaches IC2.10 (PA4)
- net ESP_EN: now also U3.3 (ON)
- net ESP_READY: now reaches IC2.11 (PA5)
- net ESP_READY: now also IC1.37 (IO41)
- net at D3.2 (A): now also J4.1 (GND); no longer SW2.1
- net GPIO_45_46: no longer names the net of IC1.41 (IO45)
- net GPIO_45_46: no longer IC1.44 (IO46)
- removed net JTAG: IC1.35 (IO39), IC1.36 (IO40), IC1.37 (IO41), IC1.38 (IO42)
- new net: IC1.33 (IO37), JP2.1 (A)
- new net: D11.2 (A), J1.2 (Pin_2)
- new net: C23.2, R31.1, SW2.2, U3.4 (IN)
- new net: D7.2 (A), J10.3 (SWCLK)
- new net: IC1.34 (IO38), JP1.1 (A)
- new net: F1.2, J1.1 (Pin_1)
- new net: D12.2 (A), J9.1, J9.2, J9.3, J9.4
- new net A_GND: J8.1, J8.2, J8.3, J8.4, JP3.2 (B)
- new net GPIO_46: IC1.44 (IO46), R41.2
- new net uCHIP_CS: IC1.14 (IO10), R36.2, R40.1
- no-connect marks 23 -> 30
Other:
- note added: "TODO Proteção: [V] Calcular valor do Diodo Zener para 3V3 [ ] proteção dos LEDS com transistor [V] proteção contra curto na fonte"
- note removed: "Debug"
- note removed: "TODO Proteção: [ ] Calcular valor do Diodo Zener para 3V3 [ ] colocar diodos para o terra em todos os componentes que têm ligação direta com o terra [ ] proteção dos LEDS com transistor [ ] proteção contra curto na fonte"
- title: Sound System - IOT -> SISTEMA DE IRRIGAÇÃO - IOT
- moved on the sheet: C11, C21, C45, C7, C8, C9, H1, H2, H3, H4, J1, J4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
